File: PCB/Main Module/modpad.kicad_sch (KiCad schematic)
At the start: 5 parts, among them J2 Bottom modular port, J4 Display Socket

Commit message: feat(Main Module): PCB v1
Parts:
- J4: footprint Connector_PinHeader_2.54mm:PinHeader_1x04_P2.54mm_Vertical -> KiCad-SSD1306-0.91-OLED-4pin-128x32.pretty-master:SSD1306-0.91-OLED-4pin-128x32
Changed lines of the file:
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@@
 			)
 		)
-		(property "Footprint" "Connector_PinHeader_2.54mm:PinHeader_1x04_P2.54mm_Vertical"
+		(property "Footprint" "KiCad-SSD1306-0.91-OLED-4pin-128x32.pretty-master:SSD1306-0.91-OLED-4pin-128x32"
 			(at 259.08 33.02 0)
 			(hide yes)
