File: PCB/Main Module/modpad.kicad_pcb (KiCad board)
At the start: 2 copper layers, 47.7 x 20 mm, 5 parts, among them J2 Bottom modular port, J4 Display Socket

Commit message: feat(Main Module): PCB v1
Parts:
- J4: footprint Connector_PinHeader_2.54mm:PinHeader_1x04_P2.54mm_Vertical -> KiCad-SSD1306-0.91-OLED-4pin-128x32.pretty-master:SSD1306-0.91-OLED-4pin-128x32
- moved J4 37.6 mm to (181.3, 41.8), turned to 180 degrees
- moved R1 4.60 mm to (141.3, 39.8), turned to -90 degrees
Connections:
- RZ1 pad 21: unconnected-(RZ1-3V3-Pad21) -> +3.3V
Routing:
- net +5V: track 0.00 -> 83.2 mm
- net SDA: track 0.00 -> 36.1 mm
- net SCL: track 0.00 -> 34.5 mm
- net INT: track 0.00 -> 34.0 mm
- net +3.3V: track 0.00 -> 30.8 mm, vias 0 -> 1
- added copper zone on B.Cu, net GND
- removed copper zone on F.Cu, net GND
Other:
- board text added: "By Ginobeano"
- board text added: "GND"
- board text added: "INT"
- board text added: "Main Module"
- board text added: "Modpad"
- board text added: "Pogo Connector"
- board text added: "SCL"
- board text added: "SDA"
- board text added: "VCC"

Commit message: feat: finish hardware designs
Routing:
- net GND: track 0.38 -> 47.2 mm
Other:
- board size 47.7 x 20 mm -> 47.7 x 20.6 mm
Changed lines of the file:
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@@
 	)
 	(gr_rect
-		(start 109.95 28.5)
-		(end 157.7 48.5)
+		(start 109.95 28.2)
+		(end 157.7 48.8)
 		(stroke
 			(width 0.05)
@@
 		(layer "F.Cu")
 		(net "INT")
-	)
-	(segment
-		(start 114.48 46.11)
-		(end 114.48 45.73)
-		(width 0.2)
-		(layer "B.Cu")
-		(net "GND")
-	)
-	(segment
-		(start 111.94 45.156856)
-		(end 122.234256 34.8626)
-		(width 2.75)
-		(layer "B.Cu")
-		(net "+5V")
-	)
-	(segment
-		(start 123.146856 33.95)
-		(end 129 33.95)
-		(width 2.75)
-		(layer "B.Cu")
-		(net "+5V")
-	)
-	(segment
-		(start 122.234256 34.8626)
-		(end 123.146856 33.95)
-		(width 2.75)
-		(layer "B.Cu")
-		(net "+5V")
-	)
-	(segment
-		(start 130.64 32.31)
-		(end 129 33.95)
-		(width 0.2)
-		(layer "B.Cu")
-		(net "+5V")
-	)
-	(segment
-		(start 137.311129 34.8626)
-		(end 122.234256 34.8626)
-		(width 0.2)
-		(layer "B.Cu")
-		(net "+5V")
-	)
-	(segment
-		(start 145.935 35.715)
-		(end 145.935 45.665)
-		(width 0.2)
-		(layer "B.Cu")
-		(net "+5V")
-	)
-	(segment
-		(start 144.785 34.565)
-		(end 145.935 35.715)
-		(width 0.2)
-		(layer "B.Cu")
-		(net "+5V")
-	)
-	(segment
-		(start 142.53 32.31)
-		(end 130.64 32.31)
-		(width 0.2)
-		(layer "B.Cu")
-		(net "+5V")
-	)
-	(segment
-		(start 144.87 42.421471)
-		(end 137.311129 34.8626)
-		(width 0.2)
-		(layer "B.Cu")
-		(net "+5V")
-	)
-	(segment
-		(start 111.94 46.11)
-		(end 111.94 45.156856)
-		(width 2.75)
-		(layer "B.Cu")
-		(net "+5V")
-	)
-	(segment
-		(start 144.785 34.565)
-		(end 142.53 32.31)
-		(width 0.2)
-		(layer "B.Cu")
-		(net "+5V")
-	)
-	(segment
-		(start 145.935 45.665)
-		(end 144.87 46.73)
-		(width 0.2)
-		(layer "B.Cu")
-		(net "+5V")
-	)
-	(segment
-		(start 144.87 46.73)
-		(end 144.87 42.421471)
-		(width 0.2)
-		(layer "B.Cu")
-		(net "+5V")
 	)
 	(segment
@@
 		(net "+3.3V")
 	)
+	(segment
+		(start 114.48 46.11)
+		(end 118.29 42.3)
+		(width 0.2)
+		(layer "F.Cu")
+		(net "GND")
+	)
+	(segment
+		(start 144.6 42.3)
+		(end 146.26 43.96)
+		(width 0.2)
+		(layer "F.Cu")
+		(net "GND")
+	)
+	(segment
+		(start 146.933654 47.88)
+		(end 153.88 47.88)
+		(width 0.2)
+		(layer "F.Cu")
+		(net "GND")
+	)
+	(segment
+		(start 146.26 43.96)
+		(end 146.26 47.206346)
+		(width 0.2)
+		(layer "F.Cu")
+		(net "GND")
+	)
+	(segment
+		(start 153.88 47.88)
+		(end 155.03 46.73)
+		(width 0.2)
+		(layer "F.Cu")
+		(net "GND")
+	)
+	(segment
+		(start 118.29 42.3)
+		(end 144.6 42.3)
+		(width 0.2)
+		(layer "F.Cu")
+		(net "GND")
+	)
+	(segment
+		(start 146.26 47.206346)
+		(end 146.933654 47.88)
+		(width 0.2)
+		(layer "F.Cu")
+		(net "GND")
+	)
+	(segment
+		(start 114.48 46.11)
+		(end 114.48 45.73)
+		(width 0.2)
+		(layer "B.Cu")
+		(net "GND")
+	)
+	(segment
+		(start 111.94 45.156856)
+		(end 122.234256 34.8626)
+		(width 2.75)
+		(layer "B.Cu")
+		(net "+5V")
+	)
+	(segment
+		(start 123.146856 33.95)
+		(end 129 33.95)
+		(width 2.75)
+		(layer "B.Cu")
+		(net "+5V")
+	)
+	(segment
+		(start 122.234256 34.8626)
+		(end 123.146856 33.95)
+		(width 2.75)
+		(layer "B.Cu")
+		(net "+5V")
+	)
+	(segment
+		(start 130.64 32.31)
+		(end 129 33.95)
+		(width 0.2)
+		(layer "B.Cu")
+		(net "+5V")
+	)
+	(segment
+		(start 137.311129 34.8626)
+		(end 122.234256 34.8626)
+		(width 0.2)
+		(layer "B.Cu")
+		(net "+5V")
+	)
+	(segment
+		(start 145.935 35.715)
+		(end 145.935 45.665)
+		(width 0.2)
+		(layer "B.Cu")
+		(net "+5V")
+	)
+	(segment
+		(start 144.785 34.565)
+		(end 145.935 35.715)
+		(width 0.2)
+		(layer "B.Cu")
+		(net "+5V")
+	)
+	(segment
+		(start 142.53 32.31)
+		(end 130.64 32.31)
+		(width 0.2)
+		(layer "B.Cu")
+		(net "+5V")
+	)
+	(segment
+		(start 144.87 42.421471)
+		(end 137.311129 34.8626)
+		(width 0.2)
+		(layer "B.Cu")
+		(net "+5V")
+	)
+	(segment
+		(start 111.94 46.11)
+		(end 111.94 45.156856)
+		(width 2.75)
+		(layer "B.Cu")
+		(net "+5V")
+	)
+	(segment
+		(start 144.785 34.565)
+		(end 142.53 32.31)
+		(width 0.2)
+		(layer "B.Cu")
+		(net "+5V")
+	)
+	(segment
+		(start 145.935 45.665)
+		(end 144.87 46.73)
+		(width 0.2)
+		(layer "B.Cu")
+		(net "+5V")
+	)
+	(segment
+		(start 144.87 46.73)
+		(end 144.87 42.421471)
+		(width 0.2)
+		(layer "B.Cu")
+		(net "+5V")
+	)
 	(zone
