File: PCB/knobs_module[/knobs_module[.kicad_sch (KiCad schematic)
At the start: 14 parts, among them J1 Conn_02x05_Odd_Even, J3 Top Modular Port, J4 Right Modular Port, J5 Left Modular Port, J6 Bottom Modular Port, U1 CH32V203F6P6, U2 XC6206PxxxMR

Commit message: feat:macro +knobs
Parts:
- added SW1, SW2: RotaryEncoder_Switch_MP, Rotary_Encoder:RotaryEncoder_Alps_EC11E-Switch_Vertical_H20mm, symbol Device:RotaryEncoder_Switch_MP
Connections:
- net GND: now also SW1.C, SW1.MP, SW2.C, SW2.MP
- net Encoder_2_A: now reaches U1.11 (PA5)
- net Encoder_2_A: now also SW2.A
- net Encoder_2_B: now reaches U1.12 (PA6)
- net Encoder_2_B: now also SW2.B
- net Encoder_1_A: now reaches U1.13 (PA7)
- net Encoder_1_A: now also SW1.A
- net Encoder_1_B: now reaches U1.14 (PB1)
- net Encoder_1_B: now also SW1.B
