File: PCB/knobs_module[/knobs_module[.kicad_pcb (KiCad board)
At the start: 2 copper layers, 80 x 80 mm, 14 parts, among them J1 Conn_02x05_Odd_Even, J3 Top Modular Port, J4 Right Modular Port, J5 Left Modular Port, J6 Bottom Modular Port, U1 CH32V203F6P6, U2 XC6206PxxxMR

Commit message: feat:macro +knobs
Parts:
- added SW1: RotaryEncoder_Switch_MP, Rotary_Encoder:RotaryEncoder_Alps_EC11E-Switch_Vertical_H20mm, F.Cu at (124.0, 104.0)
- added SW2: RotaryEncoder_Switch_MP, Rotary_Encoder:RotaryEncoder_Alps_EC11E-Switch_Vertical_H20mm, F.Cu at (163.9, 104.0)
Connections:
- U1 pad 11: unconnected-(U1-PA5-Pad11) -> Encoder_2_A
- U1 pad 12: unconnected-(U1-PA6-Pad12) -> Encoder_2_B
- U1 pad 13: unconnected-(U1-PA7-Pad13) -> Encoder_1_A
- U1 pad 14: unconnected-(U1-PB1-Pad14) -> Encoder_1_B
Routing:
- net Encoder_2_B: track 0.00 -> 56.6 mm, vias 0 -> 1
- net Encoder_2_A: track 0.00 -> 53.0 mm, vias 0 -> 1
- net Encoder_1_B: track 0.00 -> 40.1 mm, vias 0 -> 1
- net Encoder_1_A: track 0.00 -> 32.7 mm, vias 0 -> 1
- net GND: track 19.2 -> 38.8 mm

Commit message: feat: finish hardware designs
Other:
- board text added: "Modpad Knobs Module By: Ginobeano"
- board text removed: "Modpad (insert name) By: Ginobeano"
Changed lines of the file:
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@@
 		)
 		(pad_to_mask_clearance 0)
-		(solder_mask_min_width 0.12)
 		(allow_soldermask_bridges_in_footprints no)
 		(tenting
@@
 		)
 	)
-	(gr_text "Modpad (insert name)\nBy: Ginobeano"
+	(gr_text "Modpad Knobs Module\nBy: Ginobeano"
 		(at 186.85 86.4 0)
 		(layer "B.SilkS")
@@
 	)
 	(segment
+		(start 123.6 76.25)
+		(end 122.4625 76.25)
+		(width 0.127)
+		(layer "F.Cu")
+		(net "Encoder_2_A")
+	)
+	(segment
+		(start 122.4625 76.25)
+		(end 122.4375 76.275)
+		(width 0.127)
+		(layer "F.Cu")
+		(net "Encoder_2_A")
+	)
+	(via
+		(at 123.6 76.25)
+		(size 0.6)
+		(drill 0.3)
+		(layers "F.Cu" "B.Cu")
+		(net "Encoder_2_A")
+	)
+	(segment
+		(start 136.2 76.25)
+		(end 123.6 76.25)
+		(width 0.127)
+		(layer "B.Cu")
+		(net "Encoder_2_A")
+	)
+	(segment
+		(start 163.95 104)
+		(end 136.2 76.25)
+		(width 0.127)
+		(layer "B.Cu")
+		(net "Encoder_2_A")
+	)
+	(segment
+		(start 123.953152 76.925)
+		(end 122.4375 76.925)
+		(width 0.127)
+		(layer "F.Cu")
+		(net "Encoder_2_B")
+	)
+	(segment
+		(start 124.132307 76.745845)
+		(end 123.953152 76.925)
+		(width 0.127)
+		(layer "F.Cu")
+		(net "Encoder_2_B")
+	)
+	(via
+		(at 124.132307 76.745845)
+		(size 0.6)
+		(drill 0.3)
+		(layers "F.Cu" "B.Cu")
+		(net "Encoder_2_B")
+	)
+	(segment
+		(start 124.168652 76.7095)
+		(end 124.132307 76.745845)
+		(width 0.127)
+		(layer "B.Cu")
+		(net "Encoder_2_B")
+	)
+	(segment
+		(start 163.95 109)
+		(end 158.4 103.45)
+		(width 0.127)
+		(layer "B.Cu")
+		(net "Encoder_2_B")
+	)
+	(segment
+		(start 134.5095 76.7095)
+		(end 124.168652 76.7095)
+		(width 0.127)
+		(layer "B.Cu")
+		(net "Encoder_2_B")
+	)
+	(segment
+		(start 158.4 103.45)
+		(end 158.4 100.6)
+		(width 0.127)
+		(layer "B.Cu")
+		(net "Encoder_2_B")
+	)
+	(segment
+		(start 158.4 100.6)
+		(end 134.5095 76.7095)
+		(width 0.127)
+		(layer "B.Cu")
+		(net "Encoder_2_B")
+	)
+	(segment
 		(start 122.4375 77.575)
 		(end 123.910214 77.575)
@@
 		(net "Encoder_1_B")
 	)
-	(segment
-		(start 123.953152 76.925)
-		(end 122.4375 76.925)
-		(width 0.127)
-		(layer "F.Cu")
-		(net "Encoder_2_B")
-	)
-	(segment
-		(start 124.132307 76.745845)
-		(end 123.953152 76.925)
-		(width 0.127)
-		(layer "F.Cu")
-		(net "Encoder_2_B")
-	)
-	(via
-		(at 124.132307 76.745845)
-		(size 0.6)
-		(drill 0.3)
-		(layers "F.Cu" "B.Cu")
-		(net "Encoder_2_B")
-	)
-	(segment
-		(start 124.168652 76.7095)
-		(end 124.132307 76.745845)
-		(width 0.127)
-		(layer "B.Cu")
-		(net "Encoder_2_B")
-	)
-	(segment
-		(start 163.95 109)
-		(end 158.4 103.45)
-		(width 0.127)
-		(layer "B.Cu")
-		(net "Encoder_2_B")
-	)
-	(segment
-		(start 134.5095 76.7095)
-		(end 124.168652 76.7095)
-		(width 0.127)
-		(layer "B.Cu")
-		(net "Encoder_2_B")
-	)
-	(segment
-		(start 158.4 103.45)
-		(end 158.4 100.6)
-		(width 0.127)
-		(layer "B.Cu")
-		(net "Encoder_2_B")
-	)
-	(segment
-		(start 158.4 100.6)
-		(end 134.5095 76.7095)
-		(width 0.127)
-		(layer "B.Cu")
-		(net "Encoder_2_B")
-	)
-	(segment
-		(start 123.6 76.25)
-		(end 122.4625 76.25)
-		(width 0.127)
-		(layer "F.Cu")
-		(net "Encoder_2_A")
-	)
-	(segment
-		(start 122.4625 76.25)
-		(end 122.4375 76.275)
-		(width 0.127)
-		(layer "F.Cu")
-		(net "Encoder_2_A")
-	)
-	(via
-		(at 123.6 76.25)
-		(size 0.6)
-		(drill 0.3)
-		(layers "F.Cu" "B.Cu")
-		(net "Encoder_2_A")
-	)
-	(segment
-		(start 136.2 76.25)
-		(end 123.6 76.25)
-		(width 0.127)
-		(layer "B.Cu")
-		(net "Encoder_2_A")
-	)
-	(segment
-		(start 163.95 104)
-		(end 136.2 76.25)
-		(width 0.127)
-		(layer "B.Cu")
-		(net "Encoder_2_A")
-	)
 	(zone
