File: PCB/macro_module/macro_module.kicad_sch (KiCad schematic)
At the start: 14 parts, among them J1 Conn_02x05_Odd_Even, J3 Top Modular Port, J4 Right Modular Port, J5 Left Modular Port, J6 Bottom Modular Port, U1 CH32V203F6P6, U2 XC6206PxxxMR

Commit message: feat:macro +knobs
Parts:
- added SW1, SW2, SW3, SW4, SW5, SW6: SW_Push, Button_Switch_Keyboard:SW_Cherry_MX_1.00u_PCB, symbol Switch:SW_Push
Connections:
- net GND: now also SW1.2, SW2.2, SW3.2, SW4.2, SW5.2, SW6.2
- net PA5: now reaches U1.11 (PA5)
- net PA5: now also SW3.1
- net PA6: now reaches U1.12 (PA6)
- net PA6: now also SW6.1
- net PA7: now reaches U1.13 (PA7)
- net PA7: now also SW2.1
- net PB1: now reaches U1.14 (PB1)
- net PB1: now also SW5.1
- net PA11: now reaches U1.17 (PA11)
- net PA11: now also SW1.1
- net PA12: now reaches U1.18 (PA12)
- net PA12: now also SW4.1
- no-connect marks 8 -> 2

Commit message: feat: finish macro module
Parts:
- SW1, SW2, SW3, SW4, SW5, SW6: footprint Button_Switch_Keyboard:SW_Cherry_MX_1.00u_PCB -> MX_Solderable:MX-Solderable-1U
Changed lines of the file:
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@@
 			)
 		)
-		(property "Footprint" "Button_Switch_Keyboard:SW_Cherry_MX_1.00u_PCB"
+		(property "Footprint" "MX_Solderable:MX-Solderable-1U"
 			(at 110.49 128.27 0)
 			(hide yes)
@@
 			)
 		)
-		(property "Footprint" "Button_Switch_Keyboard:SW_Cherry_MX_1.00u_PCB"
+		(property "Footprint" "MX_Solderable:MX-Solderable-1U"
 			(at 154.94 114.3 0)
 			(hide yes)
@@
 			)
 		)
-		(property "Footprint" "Button_Switch_Keyboard:SW_Cherry_MX_1.00u_PCB"
+		(property "Footprint" "MX_Solderable:MX-Solderable-1U"
 			(at 110.49 114.3 0)
 			(hide yes)
@@
 			)
 		)
-		(property "Footprint" "Button_Switch_Keyboard:SW_Cherry_MX_1.00u_PCB"
+		(property "Footprint" "MX_Solderable:MX-Solderable-1U"
 			(at 132.08 114.3 0)
 			(hide yes)
@@
 			)
 		)
-		(property "Footprint" "Button_Switch_Keyboard:SW_Cherry_MX_1.00u_PCB"
+		(property "Footprint" "MX_Solderable:MX-Solderable-1U"
 			(at 132.08 128.27 0)
 			(hide yes)
@@
 			)
 		)
-		(property "Footprint" "Button_Switch_Keyboard:SW_Cherry_MX_1.00u_PCB"
+		(property "Footprint" "MX_Solderable:MX-Solderable-1U"
 			(at 154.94 128.27 0)
 			(hide yes)
