File: PCB/macro_module/macro_module.kicad_pcb (KiCad board)
At the start: 2 copper layers, 80 x 80 mm, 14 parts, among them J1 Conn_02x05_Odd_Even, J3 Top Modular Port, J4 Right Modular Port, J5 Left Modular Port, J6 Bottom Modular Port, U1 CH32V203F6P6, U2 XC6206PxxxMR

Commit message: feat: finish macro module
Parts:
- added SW1: SW_Push, MX_Solderable:MX-Solderable-1U, F.Cu at (130.8, 96.2)
- added SW2: SW_Push, MX_Solderable:MX-Solderable-1U, F.Cu at (151.2, 96.3)
- added SW3: SW_Push, MX_Solderable:MX-Solderable-1U, F.Cu at (171.6, 96.3)
- added SW4: SW_Push, MX_Solderable:MX-Solderable-1U, F.Cu at (130.8, 116.7)
- added SW5: SW_Push, MX_Solderable:MX-Solderable-1U, F.Cu at (151.2, 116.8)
- added SW6: SW_Push, MX_Solderable:MX-Solderable-1U, F.Cu at (171.6, 116.8)
Connections:
- U1 pad 11: unconnected-(U1-PA5-Pad11) -> PA5
- U1 pad 12: unconnected-(U1-PA6-Pad12) -> PA6
- U1 pad 13: unconnected-(U1-PA7-Pad13) -> PA7
- U1 pad 14: unconnected-(U1-PB1-Pad14) -> PB1
- U1 pad 17: unconnected-(U1-PA11-Pad17) -> PA11
- U1 pad 18: unconnected-(U1-PA12-Pad18) -> PA12
Routing:
- net PA6: track 0.00 -> 82.8 mm, vias 0 -> 2
- net PB1: track 0.00 -> 65.6 mm, vias 0 -> 2
- net PA5: track 0.00 -> 63.5 mm, vias 0 -> 2
- net PA7: track 0.00 -> 50.7 mm, vias 0 -> 2
- net PA12: track 0.00 -> 38.9 mm
- net PA11: track 0.00 -> 23.5 mm, vias 0 -> 2
- net GND: track 19.2 -> 22.8 mm

Commit message: feat: finish hardware designs
Other:
- board text added: "Modpad Macro Module By: Ginobeano"
- board text removed: "Modpad (insert name) By: Ginobeano"
